Commit message: Clean up repo for ROS 2 Humble: remove ROS1 artifacts, add patches and nav2
- Remove stale ROS1 .launch XML files (22 files) that can't run in ROS 2
- Remove dead backup files (*_original.py, old Kinetic Dockerfile, debug images)
- Add gazebo_ros2_control URDF-in-argv patch (fixes joint control)
- Add physics-based velocity controller and noisy odometry publisher
- Add Nav2 config and navigation launch file (SLAM + AMCL modes)
- Add world variant launch files (house, office, nao test)
- Add COLCON_IGNORE for ROS1-only packages (people, pepper_bridge, etc.)
- Translate Turkish comments to English
- Downgrade verbose INFO logging to DEBUG
- Improve .gitignore (colcon log/, ROS bags, Gazebo logs)
- Port all CMakeLists.txt and package.xml to ament/ROS 2

Co-Authored-By: Claude Opus 4.6 <noreply@anthropic.com>

File: pepper_robot/pepper_description/urdf/pepper1.0_generated_urdf/pepperGazeboCPU_no_arms.xacro (robot description, xacro)
@@ -3,108 +3,45 @@
     <!-- MACROS FOR DISABLE LINKS -->
 	<xacro:property name="PI" value="3.14159265359" />
-    <!-- <xacro:macro name="DisabledLinks" params="side side_small">
-        <plugin name="${side}Finger11_link" filename="libroboticsgroup_gazebo_disable_link_plugin.so">
-            <link>${side}Finger11_link</link>
+    <!-- GAZEBO ROS2 CONTROL -->
+    <gazebo>
+        <plugin filename="libgazebo_ros2_control.so" name="gazebo_ros2_control">
+            <parameters>$(find pepper_control)/config/pepper_ros2_controllers.yaml</parameters>
+            <ros>
+                <namespace>/</namespace>
+            </ros>
         </plugin>
-        <plugin name="${side}Finger12_link" filename="libroboticsgroup_gazebo_disable_link_plugin.so">
-            <link>${side}Finger12_link</link>
-        </plugin>
-        <plugin name="${side}Finger13_link" filename="libroboticsgroup_gazebo_disable_link_plugin.so">
-            <link>${side}Finger13_link</link>
-        </plugin>
-        <plugin name="${side}Finger21_link" filename="libroboticsgroup_gazebo_disable_link_plugin.so">
-            <link>${side}Finger21_link</link>
-        </plugin>
-        <plugin name="${side}Finger22_link" filename="libroboticsgroup_gazebo_disable_link_plugin.so">
-            <link>${side}Finger22_link</link>
-        </plugin>
-        <plugin name="${side}Finger23_link" filename="libroboticsgroup_gazebo_disable_link_plugin.so">
-            <link>${side}Finger23_link</link>
-        </plugin>
-        <plugin name="${side}Finger31_link" filename="libroboticsgroup_gazebo_disable_link_plugin.so">
-            <link>${side}Finger31_link</link>
-        </plugin>
-        <plugin name="${side}Finger32_link" filename="libroboticsgroup_gazebo_disable_link_plugin.so">
-            <link>${side}Finger32_link</link>
-        </plugin>
-        <plugin name="${side}Finger33_link" filename="libroboticsgroup_gazebo_disable_link_plugin.so">
-            <link>${side}Finger33_link</link>
-        </plugin>
-        <plugin name="${side}Finger41_link" filename="libroboticsgroup_gazebo_disable_link_plugin.so">
-            <link>${side}Finger41_link</link>
-        </plugin>
-        <plugin name="${side}Finger42_link" filename="libroboticsgroup_gazebo_disable_link_plugin.so">
-            <link>${side}Finger42_link</link>
-        </plugin>
-        <plugin name="${side}Finger43_link" filename="libroboticsgroup_gazebo_disable_link_plugin.so">
-            <link>${side}Finger43_link</link>
-        </plugin>
-        <plugin name="${side}Thumb1_link" filename="libroboticsgroup_gazebo_disable_link_plugin.so">
-            <link>${side}Thumb1_link</link>
-        </plugin>
-        <plugin name="${side}Thumb2_link" filename="libroboticsgroup_gazebo_disable_link_plugin.so">
-            <link>${side}Thumb2_link</link>
-        </plugin>
-        <plugin name="${side_small}_gripper" filename="libroboticsgroup_gazebo_disable_link_plugin.so">
-            <link>${side_small}_gripper</link>
-        </plugin>
-    </xacro:macro>  -->
-    <!-- MACROS FOR MIMIC JOINTS -->
-    <!-- Fingers -->
- <!--    <xacro:macro name="FingerMimics" params="side num">
-        <plugin name="mimic_${side}Finger${num}1" filename="libroboticsgroup_gazebo_mimic_joint_plugin.so">
-            <joint>${side}Hand</joint>
-            <mimicJoint>${side}Finger${num}1</mimicJoint>
-            <multiplier>-${PI/4}</multiplier>
-            <offset>${PI/4}</offset>
-        </plugin>
-        <plugin name="mimic_${side}Finger${num}2" filename="libroboticsgroup_gazebo_mimic_joint_plugin.so">
-            <joint>${side}Hand</joint>
-            <mimicJoint>${side}Finger${num}2</mimicJoint>
-            <multiplier>-${PI/4}</multiplier>
-            <offset>${PI/4}</offset>
-        </plugin>
-        <plugin name="mimic_${side}Finger${num}3" filename="libroboticsgroup_gazebo_mimic_joint_plugin.so">
-            <joint>${side}Hand</joint>
-            <mimicJoint>${side}Finger${num}3</mimicJoint>
-            <multiplier>-${PI/4}</multiplier>
-            <offset>${PI/4}</offset>
-        </plugin>
-    </xacro:macro>
-    <xacro:macro name="ThumbMimics" params="side">
-        <plugin name="${side}Thumb1" filename="libroboticsgroup_gazebo_mimic_joint_plugin.so">
-            <joint>${side}Hand</joint>
-            <mimicJoint>${side}Thumb1</mimicJoint>
-            <multiplier>-${PI/4}</multiplier>
-            <offset>${PI/4}</offset>
-        </plugin>
-        <plugin name="${side}Thumb2" filename="libroboticsgroup_gazebo_mimic_joint_plugin.so">
-            <joint>${side}Hand</joint>
-            <mimicJoint>${side}Thumb2</mimicJoint>
-            <multiplier>-${PI/4}</multiplier>
-            <offset>${PI/4}</offset>
-        </plugin>
-    </xacro:macro> -->
-    <!-- GAZEBO ROS CONTROL -->
-    <gazebo>
-        <plugin filename="libgazebo_ros_control.so" name="gazebo_ros_control">
-            <robotNamespace></robotNamespace>
-            <legacyModeNS>true</legacyModeNS>
-            <robotSimType>gazebo_ros_control/DefaultRobotHWSim</robotSimType>
-        </plugin>
- <!--        <xacro:FingerMimics side="L" num="1"/>
-        <xacro:FingerMimics side="L" num="2"/>
-        <xacro:FingerMimics side="L" num="3"/>
-        <xacro:FingerMimics side="L" num="4"/>
-        <xacro:FingerMimics side="R" num="1"/>
-        <xacro:FingerMimics side="R" num="2"/>
-        <xacro:FingerMimics side="R" num="3"/>
-        <xacro:FingerMimics side="R" num="4"/>
-        <xacro:ThumbMimics side="L"/>
-        <xacro:ThumbMimics side="R"/>
-        <xacro:DisabledLinks side="L" side_small="l"/>
-        <xacro:DisabledLinks side="R" side_small="r"/>  -->
-    </gazebo>
-    <!-- END OF GAZEBO ROS CONTROL PLUGIN -->
+    </gazebo>
+    <!-- END OF GAZEBO ROS2 CONTROL PLUGIN -->
+    <!-- ros2_control hardware interface block -->
+    <ros2_control name="GazeboSystem" type="system">
+        <hardware>
+            <plugin>gazebo_ros2_control/GazeboSystem</plugin>
+        </hardware>
+        <joint name="HeadYaw">
+            <command_interface name="velocity"/>
+            <state_interface name="position"><param name="initial_value">0.0</param></state_interface>
+            <state_interface name="velocity"/>
+        </joint>
+        <joint name="HeadPitch">
+            <command_interface name="velocity"/>
+            <state_interface name="position"><param name="initial_value">0.0</param></state_interface>
+            <state_interface name="velocity"/>
+        </joint>
+        <joint name="HipRoll">
+            <command_interface name="velocity"/>
+            <state_interface name="position"><param name="initial_value">0.0</param></state_interface>
+            <state_interface name="velocity"/>
+        </joint>
+        <joint name="HipPitch">
+            <command_interface name="velocity"/>
+            <state_interface name="position"><param name="initial_value">0.0</param></state_interface>
+            <state_interface name="velocity"/>
+        </joint>
+        <joint name="KneePitch">
+            <command_interface name="velocity"/>
+            <state_interface name="position"><param name="initial_value">0.0</param></state_interface>
+            <state_interface name="velocity"/>
+        </joint>
+    </ros2_control>
     <!-- GAZEBO MATERIALS -->
     <gazebo reference="base_footprint">
@@ -138,161 +75,4 @@
         <turnGravityOff>false</turnGravityOff>
     </gazebo>
-<!-- ARMS -->
-<!--     <gazebo reference="LShoulder">
-        <mu1>0.5</mu1>
-        <mu2>0.5</mu2>
-        <selfCollide>false</selfCollide>
-        <turnGravityOff>false</turnGravityOff>
-    </gazebo>
-    <gazebo reference="LBicep">
-        <mu1>0.5</mu1>
-        <mu2>0.5</mu2>
-        <selfCollide>false</selfCollide>
-        <turnGravityOff>false</turnGravityOff>
-    </gazebo>
-    <gazebo reference="LElbow">
-        <mu1>0.5</mu1>
-        <mu2>0.5</mu2>
-        <selfCollide>false</selfCollide>
-        <turnGravityOff>false</turnGravityOff>
-    </gazebo>
-    <gazebo reference="LForeArm">
-        <mu1>0.5</mu1>
-        <mu2>0.5</mu2>
-        <selfCollide>false</selfCollide>
-        <turnGravityOff>false</turnGravityOff>
-    </gazebo>
-    <gazebo reference="l_wrist">
-        <mu1>0.5</mu1>
-        <mu2>0.5</mu2>
-        <selfCollide>false</selfCollide>
-        <turnGravityOff>false</turnGravityOff>
-    </gazebo>
-    <gazebo reference="l_gripper">
-        <mu1>0.5</mu1>
-        <mu2>0.5</mu2>
-        <selfCollide>false</selfCollide>
-        <turnGravityOff>true</turnGravityOff>
-    </gazebo>
-    <gazebo reference="RShoulder">
-        <mu1>0.5</mu1>
-        <mu2>0.5</mu2>
-        <selfCollide>false</selfCollide>
-        <turnGravityOff>false</turnGravityOff>
-    </gazebo>
-    <gazebo reference="RBicep">
-        <mu1>0.5</mu1>
-        <mu2>0.5</mu2>
-        <selfCollide>false</selfCollide>
-        <turnGravityOff>false</turnGravityOff>
-    </gazebo>
-    <gazebo reference="RElbow">
-        <mu1>0.5</mu1>
-        <mu2>0.5</mu2>
-        <selfCollide>false</selfCollide>
-        <turnGravityOff>false</turnGravityOff>
-    </gazebo>
-    <gazebo reference="RForeArm">
-        <mu1>0.5</mu1>
-        <mu2>0.5</mu2>
-        <selfCollide>false</selfCollide>
-        <turnGravityOff>false</turnGravityOff>
-    </gazebo>
-    <gazebo reference="r_wrist">
-        <mu1>0.5</mu1>
-        <mu2>0.5</mu2>
-        <selfCollide>false</selfCollide>
-        <turnGravityOff>false</turnGravityOff>
-    </gazebo>
-    <gazebo reference="r_gripper">
-        <mu1>0.5</mu1>
-        <mu2>0.5</mu2>
-        <selfCollide>false</selfCollide>
-        <turnGravityOff>true</turnGravityOff>
-    </gazebo> -->
-<!--     <gazebo reference="LFinger11_link">
-        <mu1>0.5</mu1>
-        <mu2>0.5</mu2>
-        <selfCollide>false</selfCollide>
-        <turnGravityOff>true</turnGravityOff>
-    </gazebo>
-    <gazebo reference="LFinger12_link">
-        <mu1>0.5</mu1>
-        <mu2>0.5</mu2>
-        <selfCollide>false</selfCollide>
-        <turnGravityOff>true</turnGravityOff>
-    </gazebo>
-    <gazebo reference="LFinger13_link">
-        <mu1>0.5</mu1>
-        <mu2>0.5</mu2>
-        <selfCollide>false</selfCollide>
-        <turnGravityOff>true</turnGravityOff>
-    </gazebo>
-    <gazebo reference="LFinger21_link">
-        <mu1>0.5</mu1>
-        <mu2>0.5</mu2>
-        <selfCollide>false</selfCollide>
-        <turnGravityOff>true</turnGravityOff>
-    </gazebo>
-    <gazebo reference="LFinger22_link">
-        <mu1>0.5</mu1>
-        <mu2>0.5</mu2>
-        <selfCollide>false</selfCollide>
-        <turnGravityOff>true</turnGravityOff>
-    </gazebo>
-    <gazebo reference="LFinger23_link">
-        <mu1>0.5</mu1>
-        <mu2>0.5</mu2>
-        <selfCollide>false</selfCollide>
-        <turnGravityOff>true</turnGravityOff>
-    </gazebo>
-    <gazebo reference="LFinger31_link">
-        <mu1>0.5</mu1>
-        <mu2>0.5</mu2>
-        <selfCollide>false</selfCollide>
-        <turnGravityOff>true</turnGravityOff>
-    </gazebo>
-    <gazebo reference="LFinger32_link">
-        <mu1>0.5</mu1>
-        <mu2>0.5</mu2>
-        <selfCollide>false</selfCollide>
-        <turnGravityOff>true</turnGravityOff>
-    </gazebo>
-    <gazebo reference="LFinger33_link">
-        <mu1>0.5</mu1>
-        <mu2>0.5</mu2>
-        <selfCollide>false</selfCollide>
-        <turnGravityOff>true</turnGravityOff>
-    </gazebo>
-    <gazebo reference="LFinger41_link">
-        <mu1>0.5</mu1>
-        <mu2>0.5</mu2>
-        <selfCollide>false</selfCollide>
-        <turnGravityOff>true</turnGravityOff>
-    </gazebo>
-    <gazebo reference="LFinger42_link">
-        <mu1>0.5</mu1>
-        <mu2>0.5</mu2>
-        <selfCollide>false</selfCollide>
-        <turnGravityOff>true</turnGravityOff>
-    </gazebo>
-    <gazebo reference="LFinger43_link">
-        <mu1>0.5</mu1>
-        <mu2>0.5</mu2>
-        <selfCollide>false</selfCollide>
-        <turnGravityOff>true</turnGravityOff>
-    </gazebo>
-    <gazebo reference="LThumb1_link">
-        <mu1>0.5</mu1>
-        <mu2>0.5</mu2>
-        <selfCollide>false</selfCollide>
-        <turnGravityOff>true</turnGravityOff>
-    </gazebo>
-    <gazebo reference="LThumb2_link">
-        <mu1>0.5</mu1>
-        <mu2>0.5</mu2>
-        <selfCollide>false</selfCollide>
-        <turnGravityOff>true</turnGravityOff>
-    </gazebo>  -->
     <gazebo reference="Hip">
         <mu1>0.5</mu1>
@@ -343,90 +123,6 @@
         <turnGravityOff>false</turnGravityOff>
     </gazebo>
-  <!--   <gazebo reference="RFinger11_link">
-        <mu1>0.5</mu1>
-        <mu2>0.5</mu2>
-        <selfCollide>false</selfCollide>
-        <turnGravityOff>true</turnGravityOff>
-    </gazebo>
-    <gazebo reference="RFinger12_link">
-        <mu1>0.5</mu1>
-        <mu2>0.5</mu2>
-        <selfCollide>false</selfCollide>
-        <turnGravityOff>true</turnGravityOff>
-    </gazebo>
-    <gazebo reference="RFinger13_link">
-        <mu1>0.5</mu1>
-        <mu2>0.5</mu2>
-        <selfCollide>false</selfCollide>
-        <turnGravityOff>true</turnGravityOff>
-    </gazebo>
-    <gazebo reference="RFinger21_link">
-        <mu1>0.5</mu1>
-        <mu2>0.5</mu2>
-        <selfCollide>false</selfCollide>
-        <turnGravityOff>true</turnGravityOff>
-    </gazebo>
-    <gazebo reference="RFinger22_link">
-        <mu1>0.5</mu1>
-        <mu2>0.5</mu2>
-        <selfCollide>false</selfCollide>
-        <turnGravityOff>true</turnGravityOff>
-    </gazebo>
-    <gazebo reference="RFinger23_link">
-        <mu1>0.5</mu1>
-        <mu2>0.5</mu2>
-        <selfCollide>false</selfCollide>
-        <turnGravityOff>true</turnGravityOff>
-    </gazebo>
-    <gazebo reference="RFinger31_link">
-        <mu1>0.5</mu1>
-        <mu2>0.5</mu2>
-        <selfCollide>false</selfCollide>
-        <turnGravityOff>true</turnGravityOff>
-    </gazebo>
-    <gazebo reference="RFinger32_link">
-        <mu1>0.5</mu1>
-        <mu2>0.5</mu2>
-        <selfCollide>false</selfCollide>
-        <turnGravityOff>true</turnGravityOff>
-    </gazebo>
-    <gazebo reference="RFinger33_link">
-        <mu1>0.5</mu1>
-        <mu2>0.5</mu2>
-        <selfCollide>false</selfCollide>
-        <turnGravityOff>true</turnGravityOff>
-    </gazebo>
-    <gazebo reference="RFinger41_link">
-        <mu1>0.5</mu1>
-        <mu2>0.5</mu2>
-        <selfCollide>false</selfCollide>
-        <turnGravityOff>true</turnGravityOff>
-    </gazebo>
-    <gazebo reference="RFinger42_link">
-        <mu1>0.5</mu1>
-        <mu2>0.5</mu2>
-        <selfCollide>false</selfCollide>
-        <turnGravityOff>true</turnGravityOff>
-    </gazebo>
-    <gazebo reference="RFinger43_link">
-        <mu1>0.5</mu1>
-        <mu2>0.5</mu2>
-        <selfCollide>false</selfCollide>
-        <turnGravityOff>true</turnGravityOff>
-    </gazebo>
-    <gazebo reference="RThumb1_link">
-        <mu1>0.5</mu1>
-        <mu2>0.5</mu2>
-        <selfCollide>false</selfCollide>
-        <turnGravityOff>true</turnGravityOff>
-    </gazebo>
-    <gazebo reference="RThumb2_link">
-        <mu1>0.5</mu1>
-        <mu2>0.5</mu2>
-        <selfCollide>false</selfCollide>
-        <turnGravityOff>true</turnGravityOff>
-    </gazebo> -->
 <!--
-        RGB CAMERAS:
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